Commit message: Cambios brazo robot  completo

File: siro-robot/install/modelo_robot/share/modelo_robot/urdf/Seguidor_linea_robot.urdf (robot description, URDF)
Before this commit: robot Seguidor_linea_robot, 5 links, 4 joints
Joints:
- joint Eslabon_2: limit lower=-1.57 upper=1.57 effort=0 velocity=0.5 -> lower=1.57 upper=4.71 effort=0 velocity=0.5; origin xyz=20 20 28 rpy=0 0 0 -> xyz=-50 -50 -50 rpy=0 0 0

File: siro-robot/src/modelo_robot/urdf/Seguidor_linea_robot.urdf (robot description, URDF)
Before this commit: robot Seguidor_linea_robot, 5 links, 4 joints
Links:
- added link Gripper; collision mesh filename=package://modelo_robot/meshes/Ensamble_5.stl; visual mesh filename=package://modelo_robot/meshes/Ensamble_6_Pinza.stl
- added link Link_4; collision mesh filename=package://modelo_robot/meshes/Ensamble_6_Pinza.stl; visual mesh filename=package://modelo_robot/meshes/Ensamble_5.stl
Joints:
- added joint Eslabon_3: type revolute, parent Link_3, child Link_4, origin xyz=-60 122 0 rpy=0 0 0, axis 1 0 0, limit lower=3.14 upper=6.28 effort=0 velocity=0.5
- added joint Gripper_end: type revolute, parent Link_4, child Gripper, origin xyz=43 0 63 rpy=0 0 0, axis 0 0 1, limit lower=3.14 upper=6.28 effort=0 velocity=0.5
- joint Eslabon_2: limit lower=-1.57 upper=1.57 effort=0 velocity=0.5 -> lower=3.14 upper=6.28 effort=0 velocity=0.5; origin xyz=20 20 28 rpy=0 0 0 -> xyz=5 0 -125 rpy=0 0 0
